File: battlebot_schematic/battlebot_schematic.kicad_sch (KiCad schematic)
At the start: 7 parts, among them J1 ESC PWM, J2 RECEIVER, J3 ESC INPUT, J4 L298N, J5 LIPO Connection, J6 L298N Power

Commit message: circuit schematic and pcb outline
Parts:
- removed J4: L298N, Connector_PinSocket_2.54mm:PinSocket_1x06_P2.54mm_Vertical, symbol Connector_Generic:Conn_01x06
- removed J5: LIPO Connection, TerminalBlock_TE-Connectivity:TerminalBlock_TE_282834-2_1x02_P2.54mm_Horizontal, symbol Connector:Screw_Terminal_01x02
- removed J6: L298N Power, Connector_Wire:SolderWire-0.75sqmm_1x03_P4.8mm_D1.25mm_OD2.3mm, symbol Connector_Generic:Conn_01x03
- added BT1: 11.1, symbol Device:Battery_Cell
- added D1: ORANGE, symbol Device:LED
- added M1, M2: Motor_DC, symbol Motor:Motor_DC
- added R2: 220, symbol Device:R_US
- added U1: L298N, Package_TO_SOT_THT:TO-220-15_P2.54x2.54mm_StaggerOdd_Lead4.58mm_Vertical, symbol Driver_Motor:L298N
- J1: value ESC PWM -> Conn_01x03
- J2: value RECEIVER -> Conn_01x04; footprint Connector_PinSocket_2.54mm:PinSocket_1x04_P2.54mm_Vertical -> Connector_PinHeader_2.54mm:PinHeader_1x04_P2.54mm_Vertical
- J3: value ESC INPUT -> Conn_01x02; footprint TerminalBlock_TE-Connectivity:TerminalBlock_TE_282834-2_1x02_P2.54mm_Horizontal -> Connector_Wire:SolderWire-0.5sqmm_1x02_P4.6mm_D0.9mm_OD2.1mm
Connections:
- net GND: now also BT1.2 (-), D1.1 (K), U1.8 (GND)
- net at A1.10 (D7): now also U1.10 (IN3)
- net at A1.11 (D8): now also U1.7 (IN2)
- net at A1.12 (D9): now also U1.5 (IN1)
- net at A1.13 (D10): now also U1.6 (EnA)
- net at A1.16 (SCK): now also R2.2
- net at A1.7 (D4): now also U1.12 (IN4)
- net at A1.8 (D5): now also U1.11 (EnB)
- net 5V: no longer names the net of A1.27 (+5V), J1.2 (Pin_2)
- net 5V: now also U1.9 (Vss)
- net BATT+: no longer names the net of J3.2 (Pin_2)
- net BATT+: now also BT1.1 (+), U1.4 (Vs)
- net D6: no longer names the net of A1.9 (D6), J1.1 (Pin_1)
- new net: M2.1 (+), U1.13 (OUT3)
- new net: M2.2 (-), U1.14 (OUT4)
- new net: M1.1 (+), U1.2 (OUT1)
- new net: M1.2 (-), U1.3 (OUT2)
- new net: D1.2 (A), R2.1
Other:
- note added: "BUILTIN_LED"
- note added: "Left Side Motor"
- note added: "Right Side Motor"

Commit message: updated electrical diagrams
Parts:
- added M3: Brushless DC, symbol Motor:Motor_DC
Other:
- note added: "ESC"
- title: BattleBot PCB -> BattleBot Electrical Diagram
Changed lines of the file:
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@@
   (paper "A4")
   (title_block
-    (title "BattleBot PCB")
+    (title "BattleBot Electrical Diagram")
     (date "2023-11-18")
+    (rev "2")
   )
   (junction (at 138.43 132.08) (diameter 0) (color 0 0 0 0)
@@
   (junction (at 143.51 39.37) (diameter 0) (color 0 0 0 0)
   )
+  (wire (pts (xy 55.88 142.24) (xy 73.66 142.24))
+    (stroke (width 0) (type default))
+  )
   (wire (pts (xy 143.51 50.8) (xy 143.51 57.15))
     (stroke (width 0) (type default))
@@
     (stroke (width 0) (type default))
   )
+  (wire (pts (xy 55.88 140.97) (xy 55.88 142.24))
+    (stroke (width 0) (type default))
+  )
   (wire (pts (xy 138.43 143.51) (xy 138.43 132.08))
     (stroke (width 0) (type default))
@@
     (stroke (width 0) (type default))
   )
+  (wire (pts (xy 55.88 127) (xy 73.66 127))
+    (stroke (width 0) (type default))
+  )
+  (wire (pts (xy 62.23 134.62) (xy 73.66 134.62))
+    (stroke (width 0) (type default))
+  )
   (wire (pts (xy 232.41 85.09) (xy 238.76 85.09))
     (stroke (width 0) (type default))
@@
     (stroke (width 0) (type default))
   )
+  (wire (pts (xy 55.88 128.27) (xy 55.88 127))
+    (stroke (width 0) (type default))
+  )
   (wire (pts (xy 232.41 115.57) (xy 232.41 105.41))
     (stroke (width 0) (type default))
@@
     (stroke (width 0) (type default))
   )
+  (rectangle (start 187.96 137.16) (end 215.9 151.13)
+    (stroke (width 0) (type default))
+    (fill (type none))
+  )
+  (rectangle (start 128.27 41.91) (end 156.21 52.07)
+    (stroke (width 0) (type default))
+    (fill (type none))
+  )
+  (rectangle (start 73.66 120.65) (end 111.76 149.86)
+    (stroke (width 0) (type default))
+    (fill (type none))
+  )
   (text "MOTOR ESC POWER" (at 82.55 130.81 0)
     (effects (font (size 1.27 1.27)) (justify left bottom))
@@
     (effects (font (size 1.27 1.27)) (justify left bottom))
   )
+  (text "ESC" (at 90.17 120.65 0)
+    (effects (font (size 1.27 1.27)) (justify left bottom))
+  )
   (text "Left Side Motor" (at 247.65 110.49 0)
     (effects (font (size 1.27 1.27)) (justify left bottom))
@@
     (pin "1")
     (instances
-      (project "batttlebot_pcb"
+      (project "battlebot_schematic"
         (path "/2b8ae4fd-e618-49a8-a7d9-a55f2d54f1c7"
           (reference "J3") (unit 1)
@@
     (pin "2")
     (instances
-      (project "batttlebot_pcb"
+      (project "battlebot_schematic"
         (path "/2b8ae4fd-e618-49a8-a7d9-a55f2d54f1c7"
           (reference "BT1") (unit 1)
@@
     (pin "1")
     (instances
-      (project "batttlebot_pcb"
+      (project "battlebot_schematic"
         (path "/2b8ae4fd-e618-49a8-a7d9-a55f2d54f1c7"
           (reference "#PWR01") (unit 1)
@@
     (pin "3")
     (instances
-      (project "batttlebot_pcb"
+      (project "battlebot_schematic"
         (path "/2b8ae4fd-e618-49a8-a7d9-a55f2d54f1c7"
           (reference "J1") (unit 1)
@@
     (pin "4")
     (instances
-      (project "batttlebot_pcb"
+      (project "battlebot_schematic"
         (path "/2b8ae4fd-e618-49a8-a7d9-a55f2d54f1c7"
           (reference "J2") (unit 1)
@@
     )
   )
+  (symbol (lib_name "Motor_DC_1") (lib_id "Motor:Motor_DC") (at 55.88 135.89 180) (unit 1)
+    (in_bom yes) (on_board yes) (dnp no) (fields_autoplaced)
+    (property "Reference" "M3" (at 50.8 132.08 0)
+      (effects (font (size 1.27 1.27)) (justify left))
+    )
+    (property "Value" "Brushless DC" (at 50.8 134.62 0)
+      (effects (font (size 1.27 1.27)) (justify left))
+    )
+    (property "Footprint" "" (at 55.88 133.604 0)
+      (effects (font (size 1.27 1.27)) hide)
+    )
+    (property "Datasheet" "~" (at 55.88 133.604 0)
+      (effects (font (size 1.27 1.27)) hide)
+    )
+    (pin "1")
+    (pin "2")
+    (pin "3")
+    (instances
+      (project "battlebot_schematic"
+        (path "/2b8ae4fd-e618-49a8-a7d9-a55f2d54f1c7"
+          (reference "M3") (unit 1)
+        )
+      )
+    )
+  )
   (symbol (lib_id "Motor:Motor_DC") (at 238.76 107.95 0) (unit 1)
     (in_bom yes) (on_board yes) (dnp no) (fields_autoplaced)
@@
     (pin "2")
     (instances
-      (project "batttlebot_pcb"
+      (project "battlebot_schematic"
         (path "/2b8ae4fd-e618-49a8-a7d9-a55f2d54f1c7"
           (reference "M2") (unit 1)
@@
     (pin "5")
     (instances
-      (project "batttlebot_pcb"
+      (project "battlebot_schematic"
         (path "/2b8ae4fd-e618-49a8-a7d9-a55f2d54f1c7"
           (reference "U1") (unit 1)
@@
     (pin "2")
     (instances
-      (project "batttlebot_pcb"
+      (project "battlebot_schematic"
         (path "/2b8ae4fd-e618-49a8-a7d9-a55f2d54f1c7"
           (reference "M1") (unit 1)
@@
     (pin "8")
     (instances
-      (project "batttlebot_pcb"
+      (project "battlebot_schematic"
         (path "/2b8ae4fd-e618-49a8-a7d9-a55f2d54f1c7"
           (reference "A1") (unit 1)
@@
     (pin "1")
     (instances
-      (project "batttlebot_pcb"
+      (project "battlebot_schematic"
         (path "/2b8ae4fd-e618-49a8-a7d9-a55f2d54f1c7"
           (reference "#PWR02") (unit 1)
@@
     (pin "1")
     (instances
-      (project "batttlebot_pcb"
+      (project "battlebot_schematic"
         (path "/2b8ae4fd-e618-49a8-a7d9-a55f2d54f1c7"
           (reference "R2") (unit 1)
@@
     (pin "2")
     (instances
-      (project "batttlebot_pcb"
+      (project "battlebot_schematic"
         (path "/2b8ae4fd-e618-49a8-a7d9-a55f2d54f1c7"
           (reference "D1") (unit 1)
