File: batttlebot_pcb/batttlebot_pcb.kicad_sch (KiCad schematic)
At the start: 7 parts, among them J1 ESC PWM, J2 RECEIVER, J3 ESC INPUT, J4 L298N, J5 LIPO Connection, J6 L298N Power

Commit message: updated electrical diagrams
Changed lines of the file:
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@@
     (stroke (width 0) (type default))
+  )
+  (rectangle (start 179.07 57.15) (end 207.01 109.22)
+    (stroke (width 0) (type default))
+    (fill (type none))
+  )
+  (rectangle (start 78.74 119.38) (end 123.19 149.86)
+    (stroke (width 0) (type default))
+    (fill (type none))
+  )
+  (rectangle (start 129.54 40.64) (end 171.45 57.15)
+    (stroke (width 0) (type default))
+    (fill (type none))
+  )
+  (rectangle (start 189.23 137.16) (end 214.63 152.4)
+    (stroke (width 0) (type default))
+    (fill (type none))
   )
   (text "MOTOR ESC POWER" (at 82.55 130.81 0)
